Commit message: fix joint and velocity limits bug

File: share/lebai_lm3_support/urdf/lm3_macro.xacro (robot description, xacro)
@@ -35,16 +35,22 @@
 <xacro:property name="mass_link6" value="0.584"/>
 <!-- Limit of joints-->
-<xacro:property name="joint1_upper_limit" value="4" />
-<xacro:property name="joint2_upper_limit" value="4" />
-<xacro:property name="joint3_upper_limit" value="4" />
-<xacro:property name="joint4_upper_limit" value="4" />
-<xacro:property name="joint5_upper_limit" value="4" />
-<xacro:property name="joint6_upper_limit" value="4" />
-<xacro:property name="joint1_lower_limit" value="-4" />
-<xacro:property name="joint2_lower_limit" value="-4" />
-<xacro:property name="joint3_lower_limit" value="-4" />
-<xacro:property name="joint4_lower_limit" value="-4" />
-<xacro:property name="joint5_lower_limit" value="-4" />
-<xacro:property name="joint6_lower_limit" value="-4" />
+<xacro:property name="joint1_upper_limit" value="6.28" />
+<xacro:property name="joint2_upper_limit" value="6.28" />
+<xacro:property name="joint3_upper_limit" value="6.28" />
+<xacro:property name="joint4_upper_limit" value="6.28" />
+<xacro:property name="joint5_upper_limit" value="6.28" />
+<xacro:property name="joint6_upper_limit" value="6.28" />
+<xacro:property name="joint1_lower_limit" value="-6.28" />
+<xacro:property name="joint2_lower_limit" value="-6.28" />
+<xacro:property name="joint3_lower_limit" value="-6.28" />
+<xacro:property name="joint4_lower_limit" value="-6.28" />
+<xacro:property name="joint5_lower_limit" value="-6.28" />
+<xacro:property name="joint6_lower_limit" value="-6.28" />
+<xacro:property name="joint1_vel_limit" value="3.14" />
+<xacro:property name="joint2_vel_limit" value="3.14" />
+<xacro:property name="joint3_vel_limit" value="3.14" />
+<xacro:property name="joint4_vel_limit" value="3.14" />
+<xacro:property name="joint5_vel_limit" value="3.14" />
+<xacro:property name="joint6_vel_limit" value="3.14" />
 <xacro:macro name="lebai_lm3" params="prefix">
 <!-- link list -->
@@ -204,5 +210,5 @@
 	<origin xyz="0.0 0.0 ${d1}" rpy="0.0 0.0 0.0"/>
 	<axis xyz="0 0 1" />
-	<limit lower="${joint1_lower_limit}" upper="${joint1_upper_limit}" effort="100" velocity="1" />
+	<limit lower="${joint1_lower_limit}" upper="${joint1_upper_limit}" effort="100" velocity="${joint1_vel_limit}" />
 </joint>
 <joint name="${prefix}joint_2" type="revolute">
@@ -211,5 +217,5 @@
         <origin xyz="0.0 0.0 0.0" rpy="${PI_2} 0 0"/>
 	<axis xyz="0 0 1" />
-	<limit lower="${joint2_lower_limit}" upper="${joint2_upper_limit}" effort="100" velocity="1" />
+	<limit lower="${joint2_lower_limit}" upper="${joint2_upper_limit}" effort="100" velocity="${joint2_vel_limit}" />
 </joint>
 <joint name="${prefix}joint_3" type="revolute">
@@ -218,5 +224,5 @@
         <origin xyz="${a2} 0 0" rpy="0 0 0"/>
 	<axis xyz="0 0 1" />
-	<limit lower="${joint3_lower_limit}" upper="${joint3_upper_limit}" effort="100" velocity="1" />
+	<limit lower="${joint3_lower_limit}" upper="${joint3_upper_limit}" effort="100" velocity="${joint3_vel_limit}" />
 </joint>
 <joint name="${prefix}joint_4" type="revolute">
@@ -225,5 +231,5 @@
        <origin xyz="${a3} 0.0 ${d4}" rpy="0 0 0"/>
 	<axis xyz="0 0 1" />
-	<limit lower="${joint4_lower_limit}" upper="${joint4_upper_limit}" effort="100" velocity="1" />
+	<limit lower="${joint4_lower_limit}" upper="${joint4_upper_limit}" effort="100" velocity="${joint4_vel_limit}" />
 </joint>
 <joint name="${prefix}joint_5" type="revolute">
@@ -232,5 +238,5 @@
         <origin xyz="0 -${d5} 0" rpy="${PI_2} 0 0"/>
 	<axis xyz="0 0 1" />
-	<limit lower="${joint5_lower_limit}" upper="${joint5_upper_limit}" effort="5.5" velocity="1" />
+	<limit lower="${joint5_lower_limit}" upper="${joint5_upper_limit}" effort="5.5" velocity="${joint5_vel_limit}" />
 </joint>
 <joint name="${prefix}joint_6" type="revolute">
@@ -239,5 +245,5 @@
         <origin xyz="0  ${d6} 0" rpy="-${PI_2} 0 0"/>
 	<axis xyz="0 0 1" />
-	<limit lower="${joint6_lower_limit}" upper="${joint6_upper_limit}" effort="4.6" velocity="1" />
+	<limit lower="${joint6_lower_limit}" upper="${joint6_upper_limit}" effort="4.6" velocity="${joint6_vel_limit}" />
 </joint>
 <joint name="${prefix}joint_6-tool0" type="fixed">
