Commit message: add config for dual robots.

File: lebai_lm3_support/urdf/two_lm3.xacro (robot description, xacro)
@@ -2,16 +2,16 @@
 <robot xmlns:xacro="http://www.ros.org/wiki/xacro" name="lebai_lm3">
   <xacro:include filename="$(find lebai_lm3_support)/urdf/lm3_macro.xacro"/>
-  <xacro:lebai_lm3 prefix="a_"/>
-  <xacro:lebai_lm3 prefix="b_"/>
+  <xacro:lebai_lm3 prefix="robot1_"/>
+  <xacro:lebai_lm3 prefix="robot2_"/>
     <link name="world">
     </link>
-    <joint name="world_to_a" type="fixed">
+    <joint name="world_to_robot1" type="fixed">
         <parent link="world"/>
-        <child link="a_base_link"/>
+        <child link="robot1_base_link"/>
         <origin xyz="0.0 1.0 0.0" />
     </joint>
-      <joint name="world_to_b" type="fixed">
+      <joint name="world_to_robot2" type="fixed">
         <parent link="world"/>
-        <child link="b_base_link"/>
+        <child link="robot2_base_link"/>
         <origin xyz="0.0 -1.0 0.0" />
     </joint>

Commit message: Add gripper urdf file add gripper model fix bugs upadte document

File: lebai_lm3_support/urdf/two_lm3.xacro (robot description, xacro)
@@ -9,10 +9,10 @@
         <parent link="world"/>
         <child link="robot1_base_link"/>
-        <origin xyz="0.0 1.0 0.0" />
+        <origin xyz="0.0 0.5 0.0" />
     </joint>
       <joint name="world_to_robot2" type="fixed">
         <parent link="world"/>
         <child link="robot2_base_link"/>
-        <origin xyz="0.0 -1.0 0.0" />
+        <origin xyz="0.0 -0.5 0.0" />
     </joint>
 </robot>
