Commit message: fix: humble null link crash on wsl

File: lebai_lm3_support/urdf/gripper.xacro (robot description, xacro)
@@ -1,10 +1,7 @@
 <?xml version="1.0"?>
-<robot xmlns:xacro="http://www.ros.org/wiki/xacro" name="lebai_lm3">
-  	<link name="world"/>
+<!-- Note: Do NOT add a 'world' link here - it causes crashes in MoveIt Setup Assistant on WSL.
+     Instead, use a virtual_joint in the SRDF to attach the robot to the world frame. -->
+<robot xmlns:xacro="http://www.ros.org/wiki/xacro" name="lebai_gripper">
 	<xacro:include filename="$(find lebai_lm3_support)/urdf/gripper_macro.xacro"/>
   	<xacro:lebai_gripper prefix=""/>
-  	<joint name="fixed" type="fixed">
-    	<parent link="world"/>
-    	<child link="gripper_base_link"/>
-  	</joint>
 </robot>

File: lebai_lm3_support/urdf/gripper_macro.xacro (robot description, xacro)
@@ -13,12 +13,12 @@
 <xacro:property name="a3" value="-0.26"/> -->
 <!-- Robot visual and  collision dir-->
-<xacro:property name="gripper_visual_base" value="package://lebai_lm3_support/meshes/gripper/visual/gripper_base.stl" />
-<xacro:property name="gripper_visual_link1" value="package://lebai_lm3_support/meshes/gripper/visual/gripper_link1.stl" />
-<xacro:property name="gripper_visual_link2" value="package://lebai_lm3_support/meshes/gripper/visual/gripper_link2.stl" />
-<xacro:property name="gripper_visual_link_finger" value="package://lebai_lm3_support/meshes/gripper/visual/gripper_link_finger.stl" />
-<xacro:property name="gripper_collision_base" value="package://lebai_lm3_support/meshes/gripper/collision/gripper_base.stl" />
-<xacro:property name="gripper_collision_link1" value="package://lebai_lm3_support/meshes/gripper/collision/gripper_link1.stl" />
-<xacro:property name="gripper_collision_link2" value="package://lebai_lm3_support/meshes/gripper/collision/gripper_link2.stl" />
-<xacro:property name="gripper_collision_link_finger" value="package://lebai_lm3_support/meshes/gripper/collision/gripper_link_finger.stl" />
+<xacro:property name="gripper_visual_base" value="package://lebai_lm3_support/meshes/gripper/visual/gripper_base.gltf" />
+<xacro:property name="gripper_visual_link1" value="package://lebai_lm3_support/meshes/gripper/visual/gripper_link1.gltf" />
+<xacro:property name="gripper_visual_link2" value="package://lebai_lm3_support/meshes/gripper/visual/gripper_link2.gltf" />
+<xacro:property name="gripper_visual_link_finger" value="package://lebai_lm3_support/meshes/gripper/visual/gripper_link_finger.dagltfe" />
+<xacro:property name="gripper_collision_base" value="package://lebai_lm3_support/meshes/gripper/collision/gripper_base.gltf" />
+<xacro:property name="gripper_collision_link1" value="package://lebai_lm3_support/meshes/gripper/collision/gripper_link1.gltf" />
+<xacro:property name="gripper_collision_link2" value="package://lebai_lm3_support/meshes/gripper/collision/gripper_link2.gltf" />
+<xacro:property name="gripper_collision_link_finger" value="package://lebai_lm3_support/meshes/gripper/collision/gripper_link_finger.gltf" />
 <xacro:macro name="lebai_gripper" params="prefix">
 <!-- link list -->

File: lebai_lm3_support/urdf/lm3.xacro (robot description, xacro)
@@ -1,10 +1,7 @@
 <?xml version="1.0"?>
+<!-- Note: Do NOT add a 'world' link here - it causes crashes in MoveIt Setup Assistant on WSL.
+     Instead, use a virtual_joint in the SRDF to attach the robot to the world frame. -->
 <robot xmlns:xacro="http://www.ros.org/wiki/xacro" name="lebai_lm3">
-  	<link name="world"/>
 	<xacro:include filename="$(find lebai_lm3_support)/urdf/lm3_macro.xacro"/>
   	<xacro:lebai_lm3 prefix=""/>
-  	<joint name="fixed" type="fixed">
-    	<parent link="world"/>
-    	<child link="base_link"/>
-  	</joint>
 </robot>

File: lebai_lm3_support/urdf/lm3_l1.xacro (robot description, xacro)
@@ -1,10 +1,7 @@
 <?xml version="1.0"?>
+<!-- Note: Do NOT add a 'world' link here - it causes crashes in MoveIt Setup Assistant on WSL.
+     Instead, use a virtual_joint in the SRDF to attach the robot to the world frame. -->
 <robot xmlns:xacro="http://www.ros.org/wiki/xacro" name="lebai_lm3_l1">
-  	<link name="world"/>
 	<xacro:include filename="$(find lebai_lm3_support)/urdf/lm3_l1_macro.xacro"/>
   	<xacro:lebai_lm3 prefix=""/>
-  	<joint name="fixed" type="fixed">
-    	<parent link="world"/>
-    	<child link="base_link"/>
-  	</joint>
 </robot>

File: lebai_lm3_support/urdf/lm3_l1_macro.xacro (robot description, xacro)
@@ -53,16 +53,34 @@
 <xacro:property name="joint5_vel_limit" value="3.14" />
 <xacro:property name="joint6_vel_limit" value="3.14" />
-<xacro:macro name="lebai_lm3" params="prefix">
+<!-- Debug geometry sizes (used when use_simple_geometries:=true) -->
+<xacro:property name="debug_box_base" value="0.25 0.25 0.12" />
+<xacro:property name="debug_box_link1" value="0.12 0.12 0.25" />
+<xacro:property name="debug_box_link2" value="0.08 0.08 0.45" />
+<xacro:property name="debug_box_link3" value="0.07 0.07 0.40" />
+<xacro:property name="debug_box_link4" value="0.06 0.06 0.20" />
+<xacro:property name="debug_box_link5" value="0.06 0.06 0.18" />
+<xacro:property name="debug_box_link6" value="0.06 0.06 0.15" />
+<xacro:macro name="lebai_lm3" params="prefix use_simple_geometries:=false">
 <!-- link list -->
 <link name="${prefix}base_link">
 	<visual>
 		<geometry>
+			<xacro:if value="${use_simple_geometries}">
+				<box size="${debug_box_base}" />
+			</xacro:if>
+			<xacro:unless value="${use_simple_geometries}">
 			<mesh filename="${visual_base}"/>
-		</geometry>
-    	<xacro:material_white name="white"/>
-	</visual>
-	<collision>
-		<geometry>
+			</xacro:unless>
+		</geometry>
+    	<xacro:material_white name="white"/>
+	</visual>
+	<collision>
+		<geometry>
+			<xacro:if value="${use_simple_geometries}">
+				<box size="${debug_box_base}" />
+			</xacro:if>
+			<xacro:unless value="${use_simple_geometries}">
 			<mesh filename="${collision_base}" />
+			</xacro:unless>
 		</geometry>
 	</collision>
@@ -71,11 +89,21 @@
 	<visual>
 		<geometry>
+			<xacro:if value="${use_simple_geometries}">
+				<box size="${debug_box_link1}" />
+			</xacro:if>
+			<xacro:unless value="${use_simple_geometries}">
 			<mesh filename="${visual_link1}" />
-		</geometry>
-    	<xacro:material_white name="white"/>
-	</visual>
-	<collision>
-		<geometry>
+			</xacro:unless>
+		</geometry>
+    	<xacro:material_white name="white"/>
+	</visual>
+	<collision>
+		<geometry>
+			<xacro:if value="${use_simple_geometries}">
+				<box size="${debug_box_link1}" />
+			</xacro:if>
+			<xacro:unless value="${use_simple_geometries}">
 			<mesh filename="${collision_link1}" />
+			</xacro:unless>
 		</geometry>
 	</collision>
@@ -92,11 +120,21 @@
 	<visual>
 		<geometry>
+			<xacro:if value="${use_simple_geometries}">
+				<box size="${debug_box_link2}" />
+			</xacro:if>
+			<xacro:unless value="${use_simple_geometries}">
 			<mesh filename="${visual_link2}" />
-		</geometry>
-    	<xacro:material_white name="white"/>
-	</visual>
-	<collision>
-		<geometry>
+			</xacro:unless>
+		</geometry>
+    	<xacro:material_white name="white"/>
+	</visual>
+	<collision>
+		<geometry>
+			<xacro:if value="${use_simple_geometries}">
+				<box size="${debug_box_link2}" />
+			</xacro:if>
+			<xacro:unless value="${use_simple_geometries}">
 			<mesh filename="${collision_link2}" />
+			</xacro:unless>
 		</geometry>
 	</collision>
@@ -113,11 +151,21 @@
 	<visual>
 		<geometry>
+			<xacro:if value="${use_simple_geometries}">
+				<box size="${debug_box_link3}" />
+			</xacro:if>
+			<xacro:unless value="${use_simple_geometries}">
 			<mesh filename="${visual_link3}" />
-		</geometry>
-    	<xacro:material_white name="white"/>
-	</visual>
-	<collision>
-		<geometry>
+			</xacro:unless>
+		</geometry>
+    	<xacro:material_white name="white"/>
+	</visual>
+	<collision>
+		<geometry>
+			<xacro:if value="${use_simple_geometries}">
+				<box size="${debug_box_link3}" />
+			</xacro:if>
+			<xacro:unless value="${use_simple_geometries}">
 			<mesh filename="${collision_link3}" />
+			</xacro:unless>
 		</geometry>
 	</collision>
@@ -134,11 +182,21 @@
 	<visual>
 		<geometry>
+			<xacro:if value="${use_simple_geometries}">
+				<box size="${debug_box_link4}" />
+			</xacro:if>
+			<xacro:unless value="${use_simple_geometries}">
 			<mesh filename="${visual_link4}" />
-		</geometry>
-    	<xacro:material_white name="white"/>
-	</visual>
-	<collision>
-		<geometry>
+			</xacro:unless>
+		</geometry>
+    	<xacro:material_white name="white"/>
+	</visual>
+	<collision>
+		<geometry>
+			<xacro:if value="${use_simple_geometries}">
+				<box size="${debug_box_link4}" />
+			</xacro:if>
+			<xacro:unless value="${use_simple_geometries}">
 			<mesh filename="${collision_link4}" />
+			</xacro:unless>
 		</geometry>
 	</collision>
@@ -155,11 +213,21 @@
 	<visual>
 		<geometry>
+			<xacro:if value="${use_simple_geometries}">
+				<box size="${debug_box_link5}" />
+			</xacro:if>
+			<xacro:unless value="${use_simple_geometries}">
 			<mesh filename="${visual_link5}" />
-		</geometry>
-    	<xacro:material_white name="white"/>
-	</visual>
-	<collision>
-		<geometry>
+			</xacro:unless>
+		</geometry>
+    	<xacro:material_white name="white"/>
+	</visual>
+	<collision>
+		<geometry>
+			<xacro:if value="${use_simple_geometries}">
+				<box size="${debug_box_link5}" />
+			</xacro:if>
+			<xacro:unless value="${use_simple_geometries}">
 			<mesh filename="${collision_link5}" />
+			</xacro:unless>
 		</geometry>
 	</collision>
@@ -176,11 +244,21 @@
 	<visual>
 		<geometry>
+			<xacro:if value="${use_simple_geometries}">
+				<box size="${debug_box_link6}" />
+			</xacro:if>
+			<xacro:unless value="${use_simple_geometries}">
 			<mesh filename="${visual_link6}" />
-		</geometry>
-    	<xacro:material_white name="white"/>
-	</visual>
-	<collision>
-		<geometry>
+			</xacro:unless>
+		</geometry>
+    	<xacro:material_white name="white"/>
+	</visual>
+	<collision>
+		<geometry>
+			<xacro:if value="${use_simple_geometries}">
+				<box size="${debug_box_link6}" />
+			</xacro:if>
+			<xacro:unless value="${use_simple_geometries}">
 			<mesh filename="${collision_link6}" />
+			</xacro:unless>
 		</geometry>
 	</collision>
@@ -194,6 +272,23 @@
     </inertial>
 </link>
-<link name="${prefix}base" />
-<link name="${prefix}tool0"/>
+<!-- Note: Empty links crash MoveIt Setup Assistant on WSL. Adding tiny invisible geometry. -->
+<link name="${prefix}base">
+  <visual>
+    <geometry><box size="0.001 0.001 0.001"/></geometry>
+    <material name="invisible"><color rgba="0 0 0 0"/></material>
+  </visual>
+  <collision>
+    <geometry><box size="0.001 0.001 0.001"/></geometry>
+  </collision>
+</link>
+<link name="${prefix}tool0">
+  <visual>
+    <geometry><box size="0.001 0.001 0.001"/></geometry>
+    <material name="invisible"><color rgba="0 0 0 0"/></material>
+  </visual>
+  <collision>
+    <geometry><box size="0.001 0.001 0.001"/></geometry>
+  </collision>
+</link>
 <!-- end of link list -->
 <!-- joint list -->

File: lebai_lm3_support/urdf/lm3_l1_with_gripper.xacro (robot description, xacro)
@@ -1,13 +1,10 @@
 <?xml version="1.0"?>
+<!-- Note: Do NOT add a 'world' link here - it causes crashes in MoveIt Setup Assistant on WSL.
+     Instead, use a virtual_joint in the SRDF to attach the robot to the world frame. -->
 <robot xmlns:xacro="http://www.ros.org/wiki/xacro" name="lebai_lm3">
-  	<link name="world"/>
 	<xacro:include filename="$(find lebai_lm3_support)/urdf/lm3_l1_macro.xacro"/>
 	<xacro:include filename="$(find lebai_lm3_support)/urdf/gripper_macro.xacro"/>
   	<xacro:lebai_lm3 prefix=""/>
 	<xacro:lebai_gripper prefix=""/>
-  	<joint name="fixed_robot" type="fixed">
-    	<parent link="world"/>
-    	<child link="base_link"/>
-  	</joint>
   	<joint name="fixed_gripper" type="fixed">
     	<parent link="tool0"/>

File: lebai_lm3_support/urdf/lm3_macro.xacro (robot description, xacro)
@@ -53,16 +53,34 @@
 <xacro:property name="joint5_vel_limit" value="3.14" />
 <xacro:property name="joint6_vel_limit" value="3.14" />
-<xacro:macro name="lebai_lm3" params="prefix">
+<!-- Debug geometry sizes (used when use_simple_geometries:=true) -->
+<xacro:property name="debug_box_base" value="0.25 0.25 0.12" />
+<xacro:property name="debug_box_link1" value="0.12 0.12 0.25" />
+<xacro:property name="debug_box_link2" value="0.08 0.08 0.35" />
+<xacro:property name="debug_box_link3" value="0.07 0.07 0.30" />
+<xacro:property name="debug_box_link4" value="0.06 0.06 0.20" />
+<xacro:property name="debug_box_link5" value="0.06 0.06 0.18" />
+<xacro:property name="debug_box_link6" value="0.06 0.06 0.15" />
+<xacro:macro name="lebai_lm3" params="prefix use_simple_geometries:=false">
 <!-- link list -->
 <link name="${prefix}base_link">
 	<visual>
 		<geometry>
+			<xacro:if value="${use_simple_geometries}">
+				<box size="${debug_box_base}" />
+			</xacro:if>
+			<xacro:unless value="${use_simple_geometries}">
 			<mesh filename="${visual_base}"/>
-		</geometry>
-    	<xacro:material_white name="white"/>
-	</visual>
-	<collision>
-		<geometry>
+			</xacro:unless>
+		</geometry>
+    	<xacro:material_white name="white"/>
+	</visual>
+	<collision>
+		<geometry>
+			<xacro:if value="${use_simple_geometries}">
+				<box size="${debug_box_base}" />
+			</xacro:if>
+			<xacro:unless value="${use_simple_geometries}">
 			<mesh filename="${collision_base}" />
+			</xacro:unless>
 		</geometry>
 	</collision>
@@ -71,11 +89,21 @@
 	<visual>
 		<geometry>
+			<xacro:if value="${use_simple_geometries}">
+				<box size="${debug_box_link1}" />
+			</xacro:if>
+			<xacro:unless value="${use_simple_geometries}">
 			<mesh filename="${visual_link1}" />
-		</geometry>
-    	<xacro:material_white name="white"/>
-	</visual>
-	<collision>
-		<geometry>
+			</xacro:unless>
+		</geometry>
+    	<xacro:material_white name="white"/>
+	</visual>
+	<collision>
+		<geometry>
+			<xacro:if value="${use_simple_geometries}">
+				<box size="${debug_box_link1}" />
+			</xacro:if>
+			<xacro:unless value="${use_simple_geometries}">
 			<mesh filename="${collision_link1}" />
+			</xacro:unless>
 		</geometry>
 	</collision>
@@ -92,11 +120,21 @@
 	<visual>
 		<geometry>
+			<xacro:if value="${use_simple_geometries}">
+				<box size="${debug_box_link2}" />
+			</xacro:if>
+			<xacro:unless value="${use_simple_geometries}">
 			<mesh filename="${visual_link2}" />
-		</geometry>
-    	<xacro:material_white name="white"/>
-	</visual>
-	<collision>
-		<geometry>
+			</xacro:unless>
+		</geometry>
+    	<xacro:material_white name="white"/>
+	</visual>
+	<collision>
+		<geometry>
+			<xacro:if value="${use_simple_geometries}">
+				<box size="${debug_box_link2}" />
+			</xacro:if>
+			<xacro:unless value="${use_simple_geometries}">
 			<mesh filename="${collision_link2}" />
+			</xacro:unless>
 		</geometry>
 	</collision>
@@ -113,11 +151,21 @@
 	<visual>
 		<geometry>
+			<xacro:if value="${use_simple_geometries}">
+				<box size="${debug_box_link3}" />
+			</xacro:if>
+			<xacro:unless value="${use_simple_geometries}">
 			<mesh filename="${visual_link3}" />
-		</geometry>
-    	<xacro:material_white name="white"/>
-	</visual>
-	<collision>
-		<geometry>
+			</xacro:unless>
+		</geometry>
+    	<xacro:material_white name="white"/>
+	</visual>
+	<collision>
+		<geometry>
+			<xacro:if value="${use_simple_geometries}">
+				<box size="${debug_box_link3}" />
+			</xacro:if>
+			<xacro:unless value="${use_simple_geometries}">
 			<mesh filename="${collision_link3}" />
+			</xacro:unless>
 		</geometry>
 	</collision>
@@ -134,11 +182,21 @@
 	<visual>
 		<geometry>
+			<xacro:if value="${use_simple_geometries}">
+				<box size="${debug_box_link4}" />
+			</xacro:if>
+			<xacro:unless value="${use_simple_geometries}">
 			<mesh filename="${visual_link4}" />
-		</geometry>
-    	<xacro:material_white name="white"/>
-	</visual>
-	<collision>
-		<geometry>
+			</xacro:unless>
+		</geometry>
+    	<xacro:material_white name="white"/>
+	</visual>
+	<collision>
+		<geometry>
+			<xacro:if value="${use_simple_geometries}">
+				<box size="${debug_box_link4}" />
+			</xacro:if>
+			<xacro:unless value="${use_simple_geometries}">
 			<mesh filename="${collision_link4}" />
+			</xacro:unless>
 		</geometry>
 	</collision>
@@ -155,11 +213,21 @@
 	<visual>
 		<geometry>
+			<xacro:if value="${use_simple_geometries}">
+				<box size="${debug_box_link5}" />
+			</xacro:if>
+			<xacro:unless value="${use_simple_geometries}">
 			<mesh filename="${visual_link5}" />
-		</geometry>
-    	<xacro:material_white name="white"/>
-	</visual>
-	<collision>
-		<geometry>
+			</xacro:unless>
+		</geometry>
+    	<xacro:material_white name="white"/>
+	</visual>
+	<collision>
+		<geometry>
+			<xacro:if value="${use_simple_geometries}">
+				<box size="${debug_box_link5}" />
+			</xacro:if>
+			<xacro:unless value="${use_simple_geometries}">
 			<mesh filename="${collision_link5}" />
+			</xacro:unless>
 		</geometry>
 	</collision>
@@ -176,11 +244,21 @@
 	<visual>
 		<geometry>
+			<xacro:if value="${use_simple_geometries}">
+				<box size="${debug_box_link6}" />
+			</xacro:if>
+			<xacro:unless value="${use_simple_geometries}">
 			<mesh filename="${visual_link6}" />
-		</geometry>
-    	<xacro:material_white name="white"/>
-	</visual>
-	<collision>
-		<geometry>
+			</xacro:unless>
+		</geometry>
+    	<xacro:material_white name="white"/>
+	</visual>
+	<collision>
+		<geometry>
+			<xacro:if value="${use_simple_geometries}">
+				<box size="${debug_box_link6}" />
+			</xacro:if>
+			<xacro:unless value="${use_simple_geometries}">
 			<mesh filename="${collision_link6}" />
+			</xacro:unless>
 		</geometry>
 	</collision>
@@ -194,6 +272,23 @@
     </inertial>
 </link>
-<link name="${prefix}base" />
-<link name="${prefix}tool0"/>
+<!-- Note: Empty links crash MoveIt Setup Assistant on WSL. Adding tiny invisible geometry. -->
+<link name="${prefix}base">
+  <visual>
+    <geometry><box size="0.001 0.001 0.001"/></geometry>
+    <material name="invisible"><color rgba="0 0 0 0"/></material>
+  </visual>
+  <collision>
+    <geometry><box size="0.001 0.001 0.001"/></geometry>
+  </collision>
+</link>
+<link name="${prefix}tool0">
+  <visual>
+    <geometry><box size="0.001 0.001 0.001"/></geometry>
+    <material name="invisible"><color rgba="0 0 0 0"/></material>
+  </visual>
+  <collision>
+    <geometry><box size="0.001 0.001 0.001"/></geometry>
+  </collision>
+</link>
 <!-- end of link list -->
 <!-- joint list -->

File: lebai_lm3_support/urdf/lm3_with_gripper.xacro (robot description, xacro)
@@ -1,13 +1,10 @@
 <?xml version="1.0"?>
+<!-- Note: Do NOT add a 'world' link here - it causes crashes in MoveIt Setup Assistant on WSL.
+     Instead, use a virtual_joint in the SRDF to attach the robot to the world frame. -->
 <robot xmlns:xacro="http://www.ros.org/wiki/xacro" name="lebai_lm3">
-  	<link name="world"/>
 	<xacro:include filename="$(find lebai_lm3_support)/urdf/lm3_macro.xacro"/>
 	<xacro:include filename="$(find lebai_lm3_support)/urdf/gripper_macro.xacro"/>
   	<xacro:lebai_lm3 prefix=""/>
 	<xacro:lebai_gripper prefix=""/>
-  	<joint name="fixed_robot" type="fixed">
-    	<parent link="world"/>
-    	<child link="base_link"/>
-  	</joint>
   	<joint name="fixed_gripper" type="fixed">
     	<parent link="tool0"/>
