Commit message: chore: update gripper model files

File: lebai_lm3_support/urdf/gripper_macro.xacro (robot description, xacro)
@@ -13,12 +13,12 @@
 <xacro:property name="a3" value="-0.26"/> -->
 <!-- Robot visual and  collision dir-->
-<xacro:property name="gripper_visual_base" value="package://lebai_lm3_support/meshes/gripper/visual/gripper_base.gltf" />
-<xacro:property name="gripper_visual_link1" value="package://lebai_lm3_support/meshes/gripper/visual/gripper_link1.gltf" />
-<xacro:property name="gripper_visual_link2" value="package://lebai_lm3_support/meshes/gripper/visual/gripper_link2.gltf" />
-<xacro:property name="gripper_visual_link_finger" value="package://lebai_lm3_support/meshes/gripper/visual/gripper_link_finger.dagltfe" />
-<xacro:property name="gripper_collision_base" value="package://lebai_lm3_support/meshes/gripper/collision/gripper_base.gltf" />
-<xacro:property name="gripper_collision_link1" value="package://lebai_lm3_support/meshes/gripper/collision/gripper_link1.gltf" />
-<xacro:property name="gripper_collision_link2" value="package://lebai_lm3_support/meshes/gripper/collision/gripper_link2.gltf" />
-<xacro:property name="gripper_collision_link_finger" value="package://lebai_lm3_support/meshes/gripper/collision/gripper_link_finger.gltf" />
+<xacro:property name="gripper_visual_base" value="package://lebai_lm3_support/meshes/gripper/visual/gripper_base.dae" />
+<xacro:property name="gripper_visual_link1" value="package://lebai_lm3_support/meshes/gripper/visual/gripper_link1.dae" />
+<xacro:property name="gripper_visual_link2" value="package://lebai_lm3_support/meshes/gripper/visual/gripper_link2.dae" />
+<xacro:property name="gripper_visual_link_finger" value="package://lebai_lm3_support/meshes/gripper/visual/gripper_link_finger.dae" />
+<xacro:property name="gripper_collision_base" value="package://lebai_lm3_support/meshes/gripper/collision/gripper_base.dae" />
+<xacro:property name="gripper_collision_link1" value="package://lebai_lm3_support/meshes/gripper/collision/gripper_link1.dae" />
+<xacro:property name="gripper_collision_link2" value="package://lebai_lm3_support/meshes/gripper/collision/gripper_link2.dae" />
+<xacro:property name="gripper_collision_link_finger" value="package://lebai_lm3_support/meshes/gripper/collision/gripper_link_finger.dae" />
 <xacro:macro name="lebai_gripper" params="prefix">
 <!-- link list -->

Commit message: feat: model gripper passive joints with mimic

File: lebai_lm3_support/urdf/gripper_macro.xacro (robot description, xacro)
@@ -122,5 +122,5 @@
 	<origin xyz="0.025 0.0 0.0856" rpy="${PI_2} 0.0 ${PI}"/>
 	<axis xyz="0 0 1" />
-	<limit lower="-10.0" upper="10.0" effort="100" velocity="1" />
+	<limit lower="0.0" upper="${PI/3.0}" effort="100" velocity="1" />
 </joint>
 <joint name="${prefix}gripper_r_joint2" type="revolute">
@@ -129,5 +129,6 @@
         <origin xyz="0.0115 0.0 0.1056" rpy="${PI_2} 0 0"/>
 	<axis xyz="0 0 1" />
-	<limit lower="-10.0" upper="10.0" effort="100" velocity="1" />
+	<limit lower="${-PI/3.0}" upper="0.0" effort="100" velocity="1" />
+	<mimic joint="${prefix}gripper_r_joint1" multiplier="-1.0" offset="0.0" />
 </joint>
 <joint name="${prefix}gripper_r_joint_finger" type="revolute">
@@ -136,5 +137,6 @@
         <origin xyz="0.0 0.053 0.0" rpy="${PI} 0 ${PI}"/>
 	<axis xyz="0 0 1" />
-	<limit lower="-10" upper="10" effort="100" velocity="1" />
+	<limit lower="${-PI/3.0}" upper="0.0" effort="100" velocity="1" />
+	<mimic joint="${prefix}gripper_r_joint1" multiplier="-1.0" offset="0.0" />
 </joint>
 <joint name="${prefix}gripper_l_joint1" type="revolute">
@@ -143,5 +145,6 @@
 	<origin xyz="-0.025 0.0 0.0856" rpy="${PI_2} 0.0 0.0"/>
 	<axis xyz="0 0 1" />
-	<limit lower="-10.0" upper="10.0" effort="100" velocity="1" />
+	<limit lower="0.0" upper="${PI/3.0}" effort="100" velocity="1" />
+	<mimic joint="${prefix}gripper_r_joint1" multiplier="1.0" offset="0.0" />
 </joint>
 <joint name="${prefix}gripper_l_joint2" type="revolute">
@@ -150,5 +153,6 @@
         <origin xyz="-0.0115 0.0 0.1056" rpy="${PI_2} 0 ${PI}"/>
 	<axis xyz="0 0 1" />
-	<limit lower="-10.0" upper="10.0" effort="100" velocity="1" />
+	<limit lower="${-PI/3.0}" upper="0.0" effort="100" velocity="1" />
+	<mimic joint="${prefix}gripper_r_joint1" multiplier="-1.0" offset="0.0" />
 </joint>
 <joint name="${prefix}gripper_l_joint_finger" type="revolute">
@@ -157,5 +161,6 @@
         <origin xyz="0.0 0.053 0.0" rpy="${PI} 0 ${PI}"/>
 	<axis xyz="0 0 1" />
-	<limit lower="-10" upper="10" effort="100" velocity="1" />
+	<limit lower="${-PI/3.0}" upper="0.0" effort="100" velocity="1" />
+	<mimic joint="${prefix}gripper_r_joint1" multiplier="-1.0" offset="0.0" />
 </joint>
 <joint name="${prefix}gripper_joint_tip" type="fixed">

Commit message: Fix gripper tip midpoint frame

File: lebai_lm3_support/urdf/gripper_macro.xacro (robot description, xacro)
@@ -49,4 +49,5 @@
 	</collision>
 </link>
+<link name="${prefix}gripper_r_link1_end_connection" />
 <link name="${prefix}gripper_r_link2">
 	<visual>
@@ -88,4 +89,5 @@
 	</collision>
 </link>
+<link name="${prefix}gripper_l_link1_end_connection" />
 <link name="${prefix}gripper_l_link2">
 	<visual>
@@ -114,4 +116,6 @@
 	</collision>
 </link>
+<link name="${prefix}gripper_tip_midpoint_arm" />
+<link name="${prefix}gripper_tip_midpoint_counterarm" />
 <link name="${prefix}gripper_tip" />
 <!-- end of link list -->
@@ -124,4 +128,9 @@
 	<limit lower="0.0" upper="${PI/3.0}" effort="100" velocity="1" />
 </joint>
+<joint name="${prefix}gripper_r_link1_end_connection_joint" type="fixed">
+	<parent link="${prefix}gripper_r_link1"/>
+	<child link="${prefix}gripper_r_link1_end_connection"/>
+	<origin xyz="0.0 0.053 0.0" rpy="0.0 0.0 0.0"/>
+</joint>
 <joint name="${prefix}gripper_r_joint2" type="revolute">
 	<parent link="${prefix}gripper_base_link"/>
@@ -148,4 +157,9 @@
 	<mimic joint="${prefix}gripper_r_joint1" multiplier="1.0" offset="0.0" />
 </joint>
+<joint name="${prefix}gripper_l_link1_end_connection_joint" type="fixed">
+	<parent link="${prefix}gripper_l_link1"/>
+	<child link="${prefix}gripper_l_link1_end_connection"/>
+	<origin xyz="0.0 0.053 0.0" rpy="0.0 0.0 0.0"/>
+</joint>
 <joint name="${prefix}gripper_l_joint2" type="revolute">
 	<parent link="${prefix}gripper_base_link"/>
@@ -164,8 +178,27 @@
 	<mimic joint="${prefix}gripper_r_joint1" multiplier="-1.0" offset="0.0" />
 </joint>
-<joint name="${prefix}gripper_joint_tip" type="fixed">
-      <parent link="${prefix}gripper_l_link_finger"/>
-      <child link="${prefix}gripper_tip"/>
-      <origin xyz="0.0115 0.0 0.0" rpy="0.0 0.0 0.0"/>
+<joint name="${prefix}gripper_tip_midpoint_arm_joint" type="revolute">
+	<parent link="${prefix}gripper_base_link"/>
+	<child link="${prefix}gripper_tip_midpoint_arm"/>
+	<origin xyz="0.0 0.0 0.1056" rpy="0.0 0.0 0.0"/>
+	<axis xyz="0 1 0" />
+	<limit lower="${-PI}" upper="${PI}" effort="100" velocity="1" />
+	<mimic joint="${prefix}gripper_r_joint1" multiplier="1.0" offset="0.0" />
+</joint>
+<joint name="${prefix}gripper_tip_midpoint_counterarm_joint" type="revolute">
+	<parent link="${prefix}gripper_tip_midpoint_arm"/>
+	<child link="${prefix}gripper_tip_midpoint_counterarm"/>
+	<origin xyz="0.0 0.0 0.0265" rpy="0.0 0.0 0.0"/>
+	<axis xyz="0 1 0" />
+	<limit lower="${-PI}" upper="${PI}" effort="100" velocity="1" />
+	<mimic joint="${prefix}gripper_r_joint1" multiplier="-2.0" offset="0.0" />
+</joint>
+<joint name="${prefix}gripper_joint_tip" type="revolute">
+	<parent link="${prefix}gripper_tip_midpoint_counterarm"/>
+	<child link="${prefix}gripper_tip"/>
+	<origin xyz="0.0 0.0 0.0265" rpy="0.0 0.0 0.0"/>
+	<axis xyz="0 1 0" />
+	<limit lower="${-PI}" upper="${PI}" effort="100" velocity="1" />
+	<mimic joint="${prefix}gripper_r_joint1" multiplier="1.0" offset="0.0" />
 </joint>
 </xacro:macro>

Commit message: fix: add gripper finger end mimic links

File: lebai_lm3_support/urdf/gripper_macro.xacro (robot description, xacro)
@@ -76,4 +76,5 @@
 	</collision>
 </link>
+<link name="${prefix}gripper_r_link_finger_end_connection" />
 <link name="${prefix}gripper_l_link1">
 	<visual>
@@ -116,4 +117,5 @@
 	</collision>
 </link>
+<link name="${prefix}gripper_l_link_finger_end_connection" />
 <link name="${prefix}gripper_tip_midpoint_arm" />
 <link name="${prefix}gripper_tip_midpoint_counterarm" />
@@ -149,4 +151,12 @@
 	<mimic joint="${prefix}gripper_r_joint1" multiplier="-1.0" offset="0.0" />
 </joint>
+<joint name="${prefix}gripper_r_link_finger_end_connection_joint" type="revolute">
+	<parent link="${prefix}gripper_r_link_finger"/>
+	<child link="${prefix}gripper_r_link_finger_end_connection"/>
+	<origin xyz="-0.0135 -0.02 0.0" rpy="0.0 0.0 0.0"/>
+	<axis xyz="0 0 1" />
+	<limit lower="0.0" upper="${PI/3.0}" effort="100" velocity="1" />
+	<mimic joint="${prefix}gripper_r_joint1" multiplier="1.0" offset="0.0" />
+</joint>
 <joint name="${prefix}gripper_l_joint1" type="revolute">
 	<parent link="${prefix}gripper_base_link"/>
@@ -177,4 +187,12 @@
 	<limit lower="${-PI/3.0}" upper="0.0" effort="100" velocity="1" />
 	<mimic joint="${prefix}gripper_r_joint1" multiplier="-1.0" offset="0.0" />
+</joint>
+<joint name="${prefix}gripper_l_link_finger_end_connection_joint" type="revolute">
+	<parent link="${prefix}gripper_l_link_finger"/>
+	<child link="${prefix}gripper_l_link_finger_end_connection"/>
+	<origin xyz="-0.0135 -0.02 0.0" rpy="0.0 0.0 0.0"/>
+	<axis xyz="0 0 1" />
+	<limit lower="0.0" upper="${PI/3.0}" effort="100" velocity="1" />
+	<mimic joint="${prefix}gripper_r_joint1" multiplier="1.0" offset="0.0" />
 </joint>
 <joint name="${prefix}gripper_tip_midpoint_arm_joint" type="revolute">
