Commit message: fix: align controller and MoveIt joint limits
Align RSDK-007 physical URDF limits and make RSDK-011 planning overrides effective.

File: lebai_lm3_support/urdf/lm3_l1_macro.xacro (robot description, xacro)
@@ -5,4 +5,5 @@
   <xacro:include filename="$(find lebai_resources)/urdf/common_constants.xacro"/>
   <xacro:include filename="$(find lebai_resources)/urdf/common_materials.xacro"/>
+  <xacro:include filename="$(find lebai_lm3_support)/urdf/lm3_joint_limits.xacro"/>
 <!-- Robot DH parameters define joint-->
 <xacro:property name="d1" value="0.21583" />
@@ -34,23 +35,4 @@
 <xacro:property name="mass_link5" value="0.93256" />
 <xacro:property name="mass_link6" value="0.5782"/>
-<!-- Limit of joints-->
-<xacro:property name="joint1_upper_limit" value="6.28" />
-<xacro:property name="joint2_upper_limit" value="6.28" />
-<xacro:property name="joint3_upper_limit" value="6.28" />
-<xacro:property name="joint4_upper_limit" value="6.28" />
-<xacro:property name="joint5_upper_limit" value="6.28" />
-<xacro:property name="joint6_upper_limit" value="6.28" />
-<xacro:property name="joint1_lower_limit" value="-6.28" />
-<xacro:property name="joint2_lower_limit" value="-6.28" />
-<xacro:property name="joint3_lower_limit" value="-6.28" />
-<xacro:property name="joint4_lower_limit" value="-6.28" />
-<xacro:property name="joint5_lower_limit" value="-6.28" />
-<xacro:property name="joint6_lower_limit" value="-6.28" />
-<xacro:property name="joint1_vel_limit" value="3.14" />
-<xacro:property name="joint2_vel_limit" value="3.14" />
-<xacro:property name="joint3_vel_limit" value="3.14" />
-<xacro:property name="joint4_vel_limit" value="3.14" />
-<xacro:property name="joint5_vel_limit" value="3.14" />
-<xacro:property name="joint6_vel_limit" value="3.14" />
 <!-- Debug geometry sizes (used when use_simple_geometries:=true) -->
 <xacro:property name="debug_box_base" value="0.25 0.25 0.12" />

File: lebai_lm3_support/urdf/lm3_macro.xacro (robot description, xacro)
@@ -5,4 +5,5 @@
   <xacro:include filename="$(find lebai_resources)/urdf/common_constants.xacro"/>
   <xacro:include filename="$(find lebai_resources)/urdf/common_materials.xacro"/>
+  <xacro:include filename="$(find lebai_lm3_support)/urdf/lm3_joint_limits.xacro"/>
 <!-- Robot DH parameters define joint-->
 <xacro:property name="d1" value="0.21583" />
@@ -34,23 +35,4 @@
 <xacro:property name="mass_link5" value="0.969" />
 <xacro:property name="mass_link6" value="0.584"/>
-<!-- Limit of joints-->
-<xacro:property name="joint1_upper_limit" value="6.28" />
-<xacro:property name="joint2_upper_limit" value="6.28" />
-<xacro:property name="joint3_upper_limit" value="6.28" />
-<xacro:property name="joint4_upper_limit" value="6.28" />
-<xacro:property name="joint5_upper_limit" value="6.28" />
-<xacro:property name="joint6_upper_limit" value="6.28" />
-<xacro:property name="joint1_lower_limit" value="-6.28" />
-<xacro:property name="joint2_lower_limit" value="-6.28" />
-<xacro:property name="joint3_lower_limit" value="-6.28" />
-<xacro:property name="joint4_lower_limit" value="-6.28" />
-<xacro:property name="joint5_lower_limit" value="-6.28" />
-<xacro:property name="joint6_lower_limit" value="-6.28" />
-<xacro:property name="joint1_vel_limit" value="3.14" />
-<xacro:property name="joint2_vel_limit" value="3.14" />
-<xacro:property name="joint3_vel_limit" value="3.14" />
-<xacro:property name="joint4_vel_limit" value="3.14" />
-<xacro:property name="joint5_vel_limit" value="3.14" />
-<xacro:property name="joint6_vel_limit" value="3.14" />
 <!-- Debug geometry sizes (used when use_simple_geometries:=true) -->
 <xacro:property name="debug_box_base" value="0.25 0.25 0.12" />

Commit message: fix: correct LM3-L1 semantic and inertial models

File: lebai_lm3_support/urdf/lm3_l1_macro.xacro (robot description, xacro)
@@ -91,5 +91,5 @@
 	</collision>
     <inertial>
-      <origin xyz="0.0 -0.004834 -0.08972" rpy="0.0 0.0 0.0"/>
+      <origin xyz="0.0 -0.004834 -0.008972" rpy="0.0 0.0 0.0"/>
       <mass value="${mass_link1}"/>
       <inertia

File: lebai_lm3_support/urdf/lm3_l1_with_gripper.xacro (robot description, xacro)
@@ -2,5 +2,5 @@
 <!-- Note: Do NOT add a 'world' link here - it causes crashes in MoveIt Setup Assistant on WSL.
      Instead, use a virtual_joint in the SRDF to attach the robot to the world frame. -->
-<robot xmlns:xacro="http://www.ros.org/wiki/xacro" name="lebai_lm3">
+<robot xmlns:xacro="http://www.ros.org/wiki/xacro" name="lebai_lm3_l1">
 	<xacro:include filename="$(find lebai_lm3_support)/urdf/lm3_l1_macro.xacro"/>
 	<xacro:include filename="$(find lebai_lm3_support)/urdf/gripper_macro.xacro"/>

Commit message: fix: apply accepted ROS SDK review findings (#61)
* fix: constrain supported pylebai versions

* chore: remove obsolete launch surfaces

Removes obsolete launch surfaces tracked by RSDK-023 and RSDK-025.

* fix: complete workspace dependency metadata

Completes workspace dependency metadata tracked by RSDK-008 and RSDK-026.

* fix: enforce fixed arm joint names

Remove the configurable arm joint_names parameter and legacy YAML inventories. Keep the singular gripper joint parameter, reject prefixed trajectory goals, and verify fixed names across status publishing and MoveIt models.\n\nRefs: RSDK-017

* fix: propagate tutorial service failures

Route move and IO examples through one result-aware service helper. Report structured and transport failures, aggregate command outcomes, and return nonzero process exits while preserving ROS and node cleanup.\n\nRefs: RSDK-018

* feat: use standard geometry motion interfaces

Replace the custom CartesianPose message with geometry_msgs Pose and Twist contracts. Convert released SDK Euler ZYX maps strictly, normalize ROS quaternions, reject invalid geometry before SDK calls, and update examples, dependencies, tests, and docs.\n\nBREAKING CHANGE: MotionTarget and JointMotion now use geometry_msgs/Pose, SpeedLinear.velocity uses geometry_msgs/Twist, and lebai_interfaces/CartesianPose is removed.\n\nRefs: RSDK-002

* perf: publish status from bounded snapshots

Build kinematics status from one released-SDK snapshot, share aligned-rate publications, and replace per-pin IO reads with checked batch calls.

Refs: RSDK-015, RSDK-016

* fix: serialize robot initialization

Guarantee one lazy robot construction under concurrent first access and preserve retry after factory failure.

Refs: RSDK-019

* fix: validate native-bound motion and LED requests

* fix: make wait_move interruptible

* fix: enforce action goal ownership

* fix: align controller and MoveIt joint limits

Align RSDK-007 physical URDF limits and make RSDK-011 planning overrides effective.

* fix: correct LM3-L1 semantic and inertial models

* fix: namespace driver and MoveIt stacks

* fix: namespace standalone robot displays

* fix: align configuration service taxonomy

RSDK-028: move resource-list services into the config category.

RSDK-030: derive and document the complete runtime service inventory.

* docs: reconcile runtime documentation and deferred scope

RSDK-029: remove stale and unconfirmed deferred-scope claims.

RSDK-030: align user documentation with the complete runtime interface.

* ci: restore ROS linter gate

RSDK-031: gate maintained sources with reproducible copyright, flake8, and pep257 checks.

* ci: trust container workspace for linters

* ci: align flake8 operator-break policy

* test: use stable pytest plugin contracts

File: lebai_lm3_support/urdf/lm3_l1_macro.xacro (robot description, xacro)
@@ -5,4 +5,5 @@
   <xacro:include filename="$(find lebai_resources)/urdf/common_constants.xacro"/>
   <xacro:include filename="$(find lebai_resources)/urdf/common_materials.xacro"/>
+  <xacro:include filename="$(find lebai_lm3_support)/urdf/lm3_joint_limits.xacro"/>
 <!-- Robot DH parameters define joint-->
 <xacro:property name="d1" value="0.21583" />
@@ -34,23 +35,4 @@
 <xacro:property name="mass_link5" value="0.93256" />
 <xacro:property name="mass_link6" value="0.5782"/>
-<!-- Limit of joints-->
-<xacro:property name="joint1_upper_limit" value="6.28" />
-<xacro:property name="joint2_upper_limit" value="6.28" />
-<xacro:property name="joint3_upper_limit" value="6.28" />
-<xacro:property name="joint4_upper_limit" value="6.28" />
-<xacro:property name="joint5_upper_limit" value="6.28" />
-<xacro:property name="joint6_upper_limit" value="6.28" />
-<xacro:property name="joint1_lower_limit" value="-6.28" />
-<xacro:property name="joint2_lower_limit" value="-6.28" />
-<xacro:property name="joint3_lower_limit" value="-6.28" />
-<xacro:property name="joint4_lower_limit" value="-6.28" />
-<xacro:property name="joint5_lower_limit" value="-6.28" />
-<xacro:property name="joint6_lower_limit" value="-6.28" />
-<xacro:property name="joint1_vel_limit" value="3.14" />
-<xacro:property name="joint2_vel_limit" value="3.14" />
-<xacro:property name="joint3_vel_limit" value="3.14" />
-<xacro:property name="joint4_vel_limit" value="3.14" />
-<xacro:property name="joint5_vel_limit" value="3.14" />
-<xacro:property name="joint6_vel_limit" value="3.14" />
 <!-- Debug geometry sizes (used when use_simple_geometries:=true) -->
 <xacro:property name="debug_box_base" value="0.25 0.25 0.12" />
@@ -109,5 +91,5 @@
 	</collision>
     <inertial>
-      <origin xyz="0.0 -0.004834 -0.08972" rpy="0.0 0.0 0.0"/>
+      <origin xyz="0.0 -0.004834 -0.008972" rpy="0.0 0.0 0.0"/>
       <mass value="${mass_link1}"/>
       <inertia
